File: 5v_supply/5v_supply.sch (KiCad schematic (older format))
At the start: 20 parts, among them J1 B2B-XH-A, J2 BM3B-GHS, J3 B2B-XH-A, U1 LM2678SX-5.0

Commit message: changed layout to a more wide format
Parts:
- C2: footprint Capacitor_SMD:C_0805_2012Metric -> Capacitor_SMD:C_0603_1608Metric; MPN C0805C104M5RACTU -> CGA3E2X7R1H104K080AA
- C3: footprint Capacitor_SMD:C_0805_2012Metric -> Capacitor_SMD:C_0603_1608Metric; MPN CGA4C2C0G1H103J060AA -> C0603C103K3GACTU
Changed lines of the file:
@@
 F 0 "C2" H 1142 2396 50  0000 L CNN
 F 1 "100nF" H 1142 2305 50  0000 L CNN
-F 2 "Capacitor_SMD:C_0805_2012Metric" H 1050 2350 50  0001 C CNN
+F 2 "Capacitor_SMD:C_0603_1608Metric" H 1050 2350 50  0001 C CNN
 F 3 "~" H 1050 2350 50  0001 C CNN
-F 4 "C0805C104M5RACTU " H 1050 2350 50  0001 C CNN "MPN"
+F 4 "CGA3E2X7R1H104K080AA" H 1050 2350 50  0001 C CNN "MPN"
 	1    1050 2350
 	1    0    0    -1
@@
 F 0 "C3" V 2621 2050 50  0000 C CNN
 F 1 "10nF" V 2712 2050 50  0000 C CNN
-F 2 "Capacitor_SMD:C_0805_2012Metric" H 2850 2050 50  0001 C CNN
+F 2 "Capacitor_SMD:C_0603_1608Metric" H 2850 2050 50  0001 C CNN
 F 3 "~" H 2850 2050 50  0001 C CNN
-F 4 "CGA4C2C0G1H103J060AA " V 2850 2050 50  0001 C CNN "MPN"
+F 4 "C0603C103K3GACTU" V 2850 2050 50  0001 C CNN "MPN"
 	1    2850 2050
 	0    1    1    0

Commit message: replaced hall connector with pads
Parts:
- removed J2: BM3B-GHS, Connector_JST:JST_GH_BM03B-GHS-TBT_1x03-1MP_P1.25mm_Vertical, symbol Connector_Generic:Conn_01x03
- added TP1, TP2, TP3: TestPoint, TestPoint:TestPoint_THTPad_D2.0mm_Drill1.0mm, symbol Connector:TestPoint
- C1: footprint Capacitor_SMD:CP_Elec_8x10.5 -> Capacitor_SMD:CP_Elec_8x11.9; MPN EEH-ZA1E221P -> PCH1V221MCL1GS
Connections:
- net +BATT: now also TP1.1
- net GND: now also TP3.1
- net HALL_OUT: now also TP2.1
Changed lines of the file:
@@
 F 0 "C1" H 738 2396 50  0000 L CNN
 F 1 "220uF" H 738 2305 50  0000 L CNN
-F 2 "Capacitor_SMD:CP_Elec_8x10.5" H 650 2350 50  0001 C CNN
+F 2 "Capacitor_SMD:CP_Elec_8x11.9" H 650 2350 50  0001 C CNN
 F 3 "~" H 650 2350 50  0001 C CNN
-F 4 "EEH-ZA1E221P" H 650 2350 50  0001 C CNN "MPN"
+F 4 "PCH1V221MCL1GS" H 650 2350 50  0001 C CNN "MPN"
 	1    650  2350
 	1    0    0    -1
@@
 Wire Wire Line
 	1650 2250 1550 2250
-$Comp
-L Connector_Generic:Conn_01x03 J2
-U 1 1 602C2648
-P 2750 1000
-F 0 "J2" H 2668 1317 50  0000 C CNN
-F 1 "BM3B-GHS" H 2668 1226 50  0000 C CNN
-F 2 "Connector_JST:JST_GH_BM03B-GHS-TBT_1x03-1MP_P1.25mm_Vertical" H 2750 1000 50  0001 C CNN
-F 3 "~" H 2750 1000 50  0001 C CNN
-F 4 "BM3B-GHS" H 2750 1000 50  0001 C CNN "MPN"
-	1    2750 1000
-	-1   0    0    -1
-$EndComp
 Wire Wire Line
 	2950 900  3100 900
@@
 	1    0    0    -1
 $EndComp
+$Comp
+L Connector:TestPoint TP1
+U 1 1 602FFF56
+P 2950 900
+F 0 "TP1" V 3000 900 50  0000 C CNN
+F 1 "TestPoint" V 2950 1250 50  0000 C CNN
+F 2 "TestPoint:TestPoint_THTPad_D2.0mm_Drill1.0mm" H 3150 900 50  0001 C CNN
+F 3 "~" H 3150 900 50  0001 C CNN
+	1    2950 900
+	0    -1   -1   0
+$EndComp
+$Comp
+L Connector:TestPoint TP2
+U 1 1 60300698
+P 2950 1000
+F 0 "TP2" V 3000 1000 50  0000 C CNN
+F 1 "TestPoint" V 2950 1350 50  0000 C CNN
+F 2 "TestPoint:TestPoint_THTPad_D2.0mm_Drill1.0mm" H 3150 1000 50  0001 C CNN
+F 3 "~" H 3150 1000 50  0001 C CNN
+	1    2950 1000
+	0    -1   -1   0
+$EndComp
+$Comp
+L Connector:TestPoint TP3
+U 1 1 603008D3
+P 2950 1100
+F 0 "TP3" V 3000 1100 50  0000 C CNN
+F 1 "TestPoint" V 2950 1450 50  0000 C CNN
+F 2 "TestPoint:TestPoint_THTPad_D2.0mm_Drill1.0mm" H 3150 1100 50  0001 C CNN
+F 3 "~" H 3150 1100 50  0001 C CNN
+	1    2950 1100
+	0    -1   -1   0
+$EndComp
 $EndSCHEMATC

Commit message: added pcb for power connections of the motors
Parts:
- TP1, TP2, TP3: footprint TestPoint:TestPoint_THTPad_D2.0mm_Drill1.0mm -> TestPoint:TestPoint_THTPad_D1.5mm_Drill0.7mm
Changed lines of the file:
@@
 F 0 "TP1" V 3000 900 50  0000 C CNN
 F 1 "TestPoint" V 2950 1250 50  0000 C CNN
-F 2 "TestPoint:TestPoint_THTPad_D2.0mm_Drill1.0mm" H 3150 900 50  0001 C CNN
+F 2 "TestPoint:TestPoint_THTPad_D1.5mm_Drill0.7mm" H 3150 900 50  0001 C CNN
 F 3 "~" H 3150 900 50  0001 C CNN
 	1    2950 900
@@
 F 0 "TP2" V 3000 1000 50  0000 C CNN
 F 1 "TestPoint" V 2950 1350 50  0000 C CNN
-F 2 "TestPoint:TestPoint_THTPad_D2.0mm_Drill1.0mm" H 3150 1000 50  0001 C CNN
+F 2 "TestPoint:TestPoint_THTPad_D1.5mm_Drill0.7mm" H 3150 1000 50  0001 C CNN
 F 3 "~" H 3150 1000 50  0001 C CNN
 	1    2950 1000
@@
 F 0 "TP3" V 3000 1100 50  0000 C CNN
 F 1 "TestPoint" V 2950 1450 50  0000 C CNN
-F 2 "TestPoint:TestPoint_THTPad_D2.0mm_Drill1.0mm" H 3150 1100 50  0001 C CNN
+F 2 "TestPoint:TestPoint_THTPad_D1.5mm_Drill0.7mm" H 3150 1100 50  0001 C CNN
 F 3 "~" H 3150 1100 50  0001 C CNN
 	1    2950 1100
